Commit message: change model name

File: catkin_ws/src/me212bot/model/me212bot.xacro (robot description, xacro)
@@ -1,8 +1,8 @@
 <?xml version="1.0"?>
-<robot xmlns:xacro="http://www.ros.org/wiki/xacro" name="me212_robot">
+<robot xmlns:xacro="http://www.ros.org/wiki/xacro" name="me212bot">
 <link name="base_link">
     <visual>
         <geometry>
-            <mesh scale="0.001 0.001 0.001" filename="package://me212_robot/model/meshes/visual/me212_robot.stl"/>
+            <mesh scale="0.001 0.001 0.001" filename="package://me212bot/model/meshes/visual/me212bot.stl"/>
         </geometry>
         <material name="blue">
